Commit message: actualizar xacro de cobot con velocidades como parametro

File: src/clase6/robot_description/mycobot_320_m5_2022/mycobot_320_m5_2022.xacro (robot description, xacro)
@@ -150,5 +150,5 @@
   <joint name="joint1" type="revolute">
     <axis xyz="0 0 1" />
-    <limit effort="1000.0" lower="-2.93" upper="2.93" velocity="10" />
+    <limit effort="1000.0" lower="-2.93" upper="2.93" velocity="${joint_velocity}" />
     <parent link="base_link" />
     <child link="link1" />
@@ -158,5 +158,5 @@
   <joint name="joint2" type="revolute">
     <axis xyz="0 0 1" />
-    <limit effort="1000.0" lower="-2.35" upper="2.35" velocity="10" />
+    <limit effort="1000.0" lower="-2.35" upper="2.35" velocity="${joint_velocity}" />
     <parent link="link1" />
     <child link="link2" />
@@ -166,5 +166,5 @@
   <joint name="joint3" type="revolute">
     <axis xyz=" 0 0 1" />
-    <limit effort="1000.0" lower="-2.53" upper="2.53" velocity="10" />
+    <limit effort="1000.0" lower="-2.53" upper="2.53" velocity="${joint_velocity}" />
     <parent link="link2" />
     <child link="link3" />
@@ -174,5 +174,5 @@
   <joint name="joint4" type="revolute">
     <axis xyz=" 0 0 1" />
-    <limit effort="1000.0" lower="-2.53" upper="2.53" velocity="10" />
+    <limit effort="1000.0" lower="-2.53" upper="2.53" velocity="${joint_velocity}" />
     <parent link="link3" />
     <child link="link4" />
@@ -182,5 +182,5 @@
   <joint name="joint5" type="revolute">
     <axis xyz="0 0 1" />
-    <limit effort="1000.0" lower="-2.93" upper="2.93" velocity="10" />
+    <limit effort="1000.0" lower="-2.93" upper="2.93" velocity="${joint_velocity}" />
     <parent link="link4" />
     <child link="link5" />
@@ -190,5 +190,5 @@
   <joint name="joint6" type="revolute">
     <axis xyz="0 0 1" />
-    <limit effort="1000.0" lower="-3.14" upper="3.14" velocity="10" />
+    <limit effort="1000.0" lower="-3.14" upper="3.14" velocity="${joint_velocity}" />
     <parent link="link5" />
     <child link="link6" />
