Commit message: ajustar velocidades mycobot

File: src/clase5/robot_description/mycobot_320_m5_2022/mycobot_320_m5_2022.xacro (robot description, xacro)
@@ -143,5 +143,5 @@
   <joint name="joint1" type="revolute">
     <axis xyz="0 0 1" />
-    <limit effort="1000.0" lower="-2.93" upper="2.93" velocity="0" />
+    <limit effort="1000.0" lower="-2.93" upper="2.93" velocity="10" />
     <parent link="base_link" />
     <child link="link1" />
@@ -151,5 +151,5 @@
   <joint name="joint2" type="revolute">
     <axis xyz="0 0 1" />
-    <limit effort="1000.0" lower="-2.35" upper="2.35" velocity="0" />
+    <limit effort="1000.0" lower="-2.35" upper="2.35" velocity="10" />
     <parent link="link1" />
     <child link="link2" />
@@ -159,5 +159,5 @@
   <joint name="joint3" type="revolute">
     <axis xyz=" 0 0 1" />
-    <limit effort="1000.0" lower="-2.53" upper="2.53" velocity="0" />
+    <limit effort="1000.0" lower="-2.53" upper="2.53" velocity="10" />
     <parent link="link2" />
     <child link="link3" />
@@ -167,5 +167,5 @@
   <joint name="joint4" type="revolute">
     <axis xyz=" 0 0 1" />
-    <limit effort="1000.0" lower="-2.53" upper="2.53" velocity="0" />
+    <limit effort="1000.0" lower="-2.53" upper="2.53" velocity="10" />
     <parent link="link3" />
     <child link="link4" />
@@ -175,5 +175,5 @@
   <joint name="joint5" type="revolute">
     <axis xyz="0 0 1" />
-    <limit effort="1000.0" lower="-2.93" upper="2.93" velocity="0" />
+    <limit effort="1000.0" lower="-2.93" upper="2.93" velocity="10" />
     <parent link="link4" />
     <child link="link5" />
@@ -183,5 +183,5 @@
   <joint name="joint6" type="revolute">
     <axis xyz="0 0 1" />
-    <limit effort="1000.0" lower="-3.14" upper="3.14" velocity="0" />
+    <limit effort="1000.0" lower="-3.14" upper="3.14" velocity="10" />
     <parent link="link5" />
     <child link="link6" />
