Commit message: refactor

File: src/clase4/robot_description/adaptive_gripper/mycobot_adaptive_gripper.urdf (robot description, URDF)
Before this commit: robot adaptive_gripper, 7 links, 6 joints
Links:
- link gripper_base: geometry collision mesh filename=package://clase4/robot_description/adaptive_gripper/gripper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; visual mesh filename=package://clase4/robot_description/adaptive_gripper/gripper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
- link gripper_left1: geometry collision mesh filename=package://clase4/robot_description/adaptive_gripper/gripper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; visual mesh filename=package://clase4/robot_description/adaptive_gripper/gripper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
- link gripper_left2: geometry collision mesh filename=package://clase4/robot_description/adaptive_gripper/gripper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; visual mesh filename=package://clase4/robot_description/adaptive_gripper/gripper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
- link gripper_left3: geometry collision mesh filename=package://clase4/robot_description/adaptive_gripper/gripper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; visual mesh filename=package://clase4/robot_description/adaptive_gripper/gripper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
- link gripper_right1: geometry collision mesh filename=package://clase4/robot_description/adaptive_gripper/gripper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; visual mesh filename=package://clase4/robot_description/adaptive_gripper/gripper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
- link gripper_right2: geometry collision mesh filename=package://clase4/robot_description/adaptive_gripper/gripper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; visual mesh filename=package://clase4/robot_description/adaptive_gripper/gripper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
- link gripper_right3: geometry collision mesh filename=package://clase4/robot_description/adaptive_gripper/gripper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; visual mesh filename=package://clase4/robot_description/adaptive_gripper/gripper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

File: src/clase4/robot_description/mycobot_320_m5_2022/mycobot_320_m5_2022.urdf (robot description, URDF)
Before this commit: robot firefighter, 7 links, 6 joints
Links:
- link base_link: geometry collision mesh filename=package://clase4/robot_description/mycobot_320_m5_2022/base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; visual mesh filename=package://clase4/robot_description/mycobot_320_m5_2022/base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
- link link1: geometry collision mesh filename=package://clase4/robot_description/mycobot_320_m5_2022/link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; visual mesh filename=package://clase4/robot_description/mycobot_320_m5_2022/link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
- link link2: geometry collision mesh filename=package://clase4/robot_description/mycobot_320_m5_2022/link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; visual mesh filename=package://clase4/robot_description/mycobot_320_m5_2022/link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
- link link3: geometry collision mesh filename=package://clase4/robot_description/mycobot_320_m5_2022/link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; visual mesh filename=package://clase4/robot_description/mycobot_320_m5_2022/link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
- link link4: geometry collision mesh filename=package://clase4/robot_description/mycobot_320_m5_2022/link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; visual mesh filename=package://clase4/robot_description/mycobot_320_m5_2022/link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
- link link5: geometry collision mesh filename=package://clase4/robot_description/mycobot_320_m5_2022/link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; visual mesh filename=package://clase4/robot_description/mycobot_320_m5_2022/link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
- link link6: geometry collision mesh filename=package://clase4/robot_description/mycobot_320_m5_2022/link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; visual mesh filename=package://clase4/robot_description/mycobot_320_m5_2022/link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
